File: kicad/Val01.kicad_pcb (KiCad board)
At the start: 2 copper layers, 14 parts, among them U1 Pico

Commit message: update kicad
Parts:
- AnalogOutPin1, LogInPin1, LogInPin2, NeoPixelInPin1: footprint Button_Switch_SMD:SW_SPST_B3U-1000P-B -> Button_Switch_THT:SW_PUSH_6mm
- LogOutPin1: footprint LED_SMD:LED_0603_1608Metric -> LED_THT:LED_D3.0mm
- LogR1: renamed from R4; footprint Resistor_SMD:R_0603_1608Metric -> Resistor_THT:R_Axial_DIN0207_L6.3mm_D2.5mm_P15.24mm_Horizontal
- LogR2: renamed from R2; footprint Resistor_SMD:R_0603_1608Metric -> Resistor_THT:R_Axial_DIN0207_L6.3mm_D2.5mm_P15.24mm_Horizontal
- LogR3: renamed from R3; footprint Resistor_SMD:R_0603_1608Metric -> Resistor_THT:R_Axial_DIN0207_L6.3mm_D2.5mm_P15.24mm_Horizontal
- LogR4: renamed from R1; footprint Resistor_SMD:R_0603_1608Metric -> Resistor_THT:R_Axial_DIN0207_L6.3mm_D2.5mm_P15.24mm_Horizontal
- LogR5: renamed from R5; footprint Resistor_SMD:R_0603_1608Metric -> Resistor_THT:R_Axial_DIN0207_L6.3mm_D2.5mm_P15.24mm_Horizontal
- NeoPixelR1: renamed from R7; footprint Resistor_SMD:R_0603_1608Metric -> Resistor_THT:R_Axial_DIN0207_L6.3mm_D2.5mm_P15.24mm_Horizontal
- NeoPixelR2: renamed from R6; footprint Resistor_SMD:R_0603_1608Metric -> Resistor_THT:R_Axial_DIN0207_L6.3mm_D2.5mm_P15.24mm_Horizontal
- moved LogR1 113.0 mm to (21.7, 25.4), turned to -90 degrees
- moved NeoPixelR2 69.2 mm to (127.0, 71.1), turned to 90 degrees
- moved LogR3 60.2 mm to (22.9, 64.1), turned to 90 degrees
- moved NeoPixelR1 59.7 mm to (127.0, 48.3), turned to 90 degrees
- moved AnalogInPin1 58.0 mm to (114.2, 36.5), turned to -90 degrees
- moved NeoPixelInPin1 47.4 mm to (105.3, 56.5)
- moved LogR2 30.9 mm to (52.2, 38.1), turned to 90 degrees
- moved LogInPin1 28.8 mm to (39.5, 27.4), turned to 180 degrees
- moved AnalogOutPin1 28.0 mm to (36.7, 76.2)
- moved LogR4 25.7 mm to (50.8, 48.8), turned to -90 degrees
- moved U1 25.7 mm to (81.3, 48.3)
- moved LogOutPin1 19.5 mm to (63.5, 61.0), turned to 180 degrees
- moved LogInPin2 14.8 mm to (31.6, 59.0)
- moved LogR5 14.4 mm to (61.0, 35.6), turned to -90 degrees
Connections:
- U1 pad 18: unconnected-(U1-GND-Pad18) -> GND
- U1 pad 23: unconnected-(U1-GND-Pad23) -> GND
- U1 pad 28: unconnected-(U1-GND-Pad28) -> GND
- U1 pad 3: unconnected-(U1-GND-Pad3) -> GND
Routing:
- net GND: track 0.00 -> 155.9 mm
- net +3V0: track 0.00 -> 145.5 mm
- net Net-(AnalogOutPin1--): track 0.00 -> 37.6 mm
- net Net-(U1-GPIO16): track 0.00 -> 37.4 mm
- net Net-(U1-GPIO1): track 0.00 -> 35.9 mm
- net Net-(U1-GPIO0): track 0.00 -> 26.0 mm
- net Net-(U1-GPIO26_ADC0): track 0.00 -> 25.2 mm
- net Net-(LogInPin1-Pad2): track 0.00 -> 25.0 mm
- net Net-(LogInPin2-Pad2): track 0.00 -> 21.9 mm
- net Net-(NeoPixelInPin1-Pad2): track 0.00 -> 17.3 mm
- net Net-(U1-GPIO2): track 0.00 -> 13.0 mm
- net Net-(LogOutPin1-A): track 0.00 -> 10.2 mm
