File: kicad/Val01.kicad_sch (KiCad schematic)
At the start: 14 parts, among them U1 Pico

Commit message: update kicad
Parts:
- AnalogOutPin1, LogInPin1, LogInPin2, NeoPixelInPin1: footprint Button_Switch_SMD:SW_SPST_B3U-1000P-B -> Button_Switch_THT:SW_PUSH_6mm
- LogOutPin1: footprint LED_SMD:LED_0603_1608Metric -> LED_THT:LED_D3.0mm
- LogR1: renamed from R4; footprint Resistor_SMD:R_0603_1608Metric -> Resistor_THT:R_Axial_DIN0207_L6.3mm_D2.5mm_P15.24mm_Horizontal
- LogR2: renamed from R2; footprint Resistor_SMD:R_0603_1608Metric -> Resistor_THT:R_Axial_DIN0207_L6.3mm_D2.5mm_P15.24mm_Horizontal
- LogR3: renamed from R3; footprint Resistor_SMD:R_0603_1608Metric -> Resistor_THT:R_Axial_DIN0207_L6.3mm_D2.5mm_P15.24mm_Horizontal
- LogR4: renamed from R1; footprint Resistor_SMD:R_0603_1608Metric -> Resistor_THT:R_Axial_DIN0207_L6.3mm_D2.5mm_P15.24mm_Horizontal
- LogR5: renamed from R5; footprint Resistor_SMD:R_0603_1608Metric -> Resistor_THT:R_Axial_DIN0207_L6.3mm_D2.5mm_P15.24mm_Horizontal
- NeoPixelR1: renamed from R7; footprint Resistor_SMD:R_0603_1608Metric -> Resistor_THT:R_Axial_DIN0207_L6.3mm_D2.5mm_P15.24mm_Horizontal
- NeoPixelR2: renamed from R6; footprint Resistor_SMD:R_0603_1608Metric -> Resistor_THT:R_Axial_DIN0207_L6.3mm_D2.5mm_P15.24mm_Horizontal
Connections:
- net GND: now also U1.18 (GND), U1.23 (GND), U1.28 (GND), U1.3 (GND)
